Commit message: Add cmd_vel bridge and config correct param for nav2

File: install/x500_bridge/share/x500_bridge/urdf/x500_lidar.urdf.xacro (robot description, xacro)
@@ -1 +1,47 @@
-/home/imamalghifary/ws_sensor_combined/build/x500_bridge/urdf/x500_lidar.urdf.xacro
+<?xml version="1.0"?>
+<robot name="x500_lidar" xmlns:xacro="http://ros.org/wiki/xacro">
+  <!-- Base footprint (at ground contact) -->
+  <link name="base_footprint"/>
+  <!-- Base link (main body of the drone) -->
+  <link name="base_link">
+    <visual>
+      <geometry>
+        <box size="0.3 0.3 0.1"/> <!-- simple placeholder -->
+      </geometry>
+      <material name="gray">
+        <color rgba="0.5 0.5 0.5 1.0"/>
+      </material>
+    </visual>
+  </link>
+  <!-- Fixed joint between base_footprint and base_link -->
+  <joint name="base_footprint_joint" type="fixed">
+    <parent link="base_footprint"/>
+    <child link="base_link"/>
+    <origin xyz="0 0 0.1" rpy="0 0 0"/> <!-- adjust height if needed -->
+  </joint>
+  <!-- LiDAR link -->
+  <link name="lidar_link">
+    <visual>
+      <geometry>
+        <cylinder radius="0.05" length="0.1"/> <!-- simplified lidar shape -->
+      </geometry>
+      <material name="blue">
+        <color rgba="0 0 1 1.0"/>
+      </material>
+    </visual>
+  </link>
+  <!-- LiDAR joint: place relative to base_link -->
+  <joint name="lidar_joint" type="fixed">
+    <parent link="base_link"/>
+    <child link="lidar_link"/>
+    <!-- From your SDF: lidar pose ≈ -0.1 0 0.26 -->
+    <origin xyz="-0.1 0 0.26" rpy="0 0 0"/>
+  </joint>
+  <!-- Odometry frame -->
+  <!-- <link name="odom"/>
+  <joint name="odom_to_base" type="fixed">
+    <parent link="odom"/>
+    <child link="base_footprint"/>
+    <origin xyz="0 0 0" rpy="0 0 0"/>
+  </joint> -->
+</robot>

Commit message: Complete Mapping, Navigation, and BT Setup

File: install/x500_bridge/share/x500_bridge/urdf/x500_lidar.urdf.xacro (robot description, xacro)
@@ -1,47 +1 @@
-<?xml version="1.0"?>
-<robot name="x500_lidar" xmlns:xacro="http://ros.org/wiki/xacro">
-  <!-- Base footprint (at ground contact) -->
-  <link name="base_footprint"/>
-  <!-- Base link (main body of the drone) -->
-  <link name="base_link">
-    <visual>
-      <geometry>
-        <box size="0.3 0.3 0.1"/> <!-- simple placeholder -->
-      </geometry>
-      <material name="gray">
-        <color rgba="0.5 0.5 0.5 1.0"/>
-      </material>
-    </visual>
-  </link>
-  <!-- Fixed joint between base_footprint and base_link -->
-  <joint name="base_footprint_joint" type="fixed">
-    <parent link="base_footprint"/>
-    <child link="base_link"/>
-    <origin xyz="0 0 0.1" rpy="0 0 0"/> <!-- adjust height if needed -->
-  </joint>
-  <!-- LiDAR link -->
-  <link name="lidar_link">
-    <visual>
-      <geometry>
-        <cylinder radius="0.05" length="0.1"/> <!-- simplified lidar shape -->
-      </geometry>
-      <material name="blue">
-        <color rgba="0 0 1 1.0"/>
-      </material>
-    </visual>
-  </link>
-  <!-- LiDAR joint: place relative to base_link -->
-  <joint name="lidar_joint" type="fixed">
-    <parent link="base_link"/>
-    <child link="lidar_link"/>
-    <!-- From your SDF: lidar pose ≈ -0.1 0 0.26 -->
-    <origin xyz="-0.1 0 0.26" rpy="0 0 0"/>
-  </joint>
-  <!-- Odometry frame -->
-  <!-- <link name="odom"/>
-  <joint name="odom_to_base" type="fixed">
-    <parent link="odom"/>
-    <child link="base_footprint"/>
-    <origin xyz="0 0 0" rpy="0 0 0"/>
-  </joint> -->
-</robot>
+/home/imamalghifary/ws_sensor_combined/build/x500_bridge/urdf/x500_lidar.urdf.xacro
